File: board/iceBlinkPico/iceblink.kicad_pcb (KiCad board)
At the start: 4 copper layers, 50.8 x 20.3 mm, 57 parts, among them J1 USB4105-GF-A, J2 Left, J3 Right, U1 W25Q128JV, U2 MIC5365-1-2YD5, U3 MIC5318-3-3YD5, U4 ICE40UP5K-SG48ITR, X1 IQXO-791

Commit message: Update to PCB to fix LED current limiting resistor values.
Parts:
- R8: value 1.5K -> 1K
- R9: value 1K -> 5.1K
